Commit message: Don't use world frame in moveit

File: interbotix_moveit/config/srdf/px100.srdf.xacro (robot description, xacro)
@@ -17,5 +17,4 @@
         <joint name="wrist_angle" />
         <joint name="ee_arm" />
-        <joint name="fixed" />
     </group>
     <group name="interbotix_gripper">

File: interbotix_moveit/config/srdf/px150.srdf.xacro (robot description, xacro)
@@ -18,5 +18,4 @@
         <joint name="wrist_rotate" />
         <joint name="ee_arm" />
-        <joint name="fixed" />
     </group>
     <group name="interbotix_gripper">

File: interbotix_moveit/config/srdf/rx150.srdf.xacro (robot description, xacro)
@@ -18,5 +18,4 @@
         <joint name="wrist_rotate" />
         <joint name="ee_arm" />
-        <joint name="fixed" />
     </group>
     <group name="interbotix_gripper">

File: interbotix_moveit/config/srdf/rx200.srdf.xacro (robot description, xacro)
@@ -18,5 +18,4 @@
         <joint name="wrist_rotate" />
         <joint name="ee_arm" />
-        <joint name="fixed" />
     </group>
     <group name="interbotix_gripper">

File: interbotix_moveit/config/srdf/vx250.srdf.xacro (robot description, xacro)
@@ -18,5 +18,4 @@
         <joint name="wrist_rotate" />
         <joint name="ee_arm" />
-        <joint name="fixed" />
     </group>
     <group name="interbotix_gripper">

File: interbotix_moveit/config/srdf/vx300.srdf.xacro (robot description, xacro)
@@ -12,5 +12,4 @@
     <xacro:arg name="robot_name" default=""/>
     <group name="interbotix_arm">
-        <joint name="fixed" />
         <joint name="waist" />
         <joint name="shoulder" />

File: interbotix_moveit/config/srdf/vx300s.srdf.xacro (robot description, xacro)
@@ -12,5 +12,4 @@
     <xacro:arg name="robot_name" default=""/>
     <group name="interbotix_arm">
-        <joint name="fixed" />
         <joint name="waist" />
         <joint name="shoulder" />

File: interbotix_moveit/config/srdf/wx200.srdf.xacro (robot description, xacro)
@@ -12,5 +12,4 @@
     <xacro:arg name="robot_name" default=""/>
     <group name="interbotix_arm">
-        <joint name="fixed" />
         <joint name="waist" />
         <joint name="shoulder" />

File: interbotix_moveit/config/srdf/wx250.srdf.xacro (robot description, xacro)
@@ -12,5 +12,4 @@
     <xacro:arg name="robot_name" default=""/>
     <group name="interbotix_arm">
-        <joint name="fixed" />
         <joint name="waist" />
         <joint name="shoulder" />

File: interbotix_moveit/config/srdf/wx250s.srdf.xacro (robot description, xacro)
@@ -12,5 +12,4 @@
     <xacro:arg name="robot_name" default=""/>
     <group name="interbotix_arm">
-        <joint name="fixed" />
         <joint name="waist" />
         <joint name="shoulder" />
